Commit message: Updated a lot of stuff: Got URDFs working in RViz & Gazebo, improved launch files, added .stl files for armbot_1.

File: src/armbot_1/urdf/arm1.xacro (robot description, xacro)
@@ -1,263 +1,322 @@
 <?xml version="1.0"?>
 <robot name="arm1" xmlns:xacro="http://www.ros.org/wiki/xacro">
+<xacro:property name="base_link_mass" value="0.1"/>
+<xacro:property name="base_link_length" value="0.05"/>
+<xacro:property name="base_link_width" value="0.05"/>
+<xacro:property name="base_link_height" value="0.05"/>
 <xacro:property name="arm_link_radius" value="0.017"/>
 <xacro:property name="arm_link_len" value="0.04"/>
+<xacro:property name="link_mass" value="0.025"/>
+<xacro:property name="head_link_mass" value="0.025"/>
+<xacro:property name="head_link_length" value="0.017"/>
+<xacro:property name="head_link_width" value="0.094"/>
+<xacro:property name="head_link_height" value="0.04"/>
+<xacro:property name="gripper_mass" value="0.01"/>
+<!--Intertial Macros-->
+<xacro:macro name="arm_base_inertial" params="mass">
+    <inertial>
+        <mass value="${base_link_mass}"/>
+        <inertia ixx="0.000041667" ixy="0" ixz="0"
+                iyy="0.000041667" iyz="0"
+                izz="0.000041667"/>
+        </inertial>
+</xacro:macro>
+<xacro:macro name="link_inertial" params="mass">
+    <inertial>
+        <mass value="${link_mass}"/>
+        <inertia ixx="0.000010279" ixy="0" ixz="0"
+                iyy="0.000010279" iyz="0"
+                izz="0.000007225"/>
+        </inertial>
+</xacro:macro>
+.000010279
+<xacro:macro name="gripper_inertial" params="mass">
+    <inertial>
+        <mass value="${gripper_mass}"/>
+        <inertia ixx="0.001" ixy="0" ixz="0"
+                iyy="0.001" iyz="0"
+                izz="0.001"/>
+        </inertial>
+</xacro:macro>
+<!--Base Link-->
+    <link name="base_link"></link>
+    <joint name="base_to_arm_base" type="fixed">
+        <parent link="base_link"/>
+        <child link="arm_base_link"/>
+        <origin xyz="0 0 0" rpy="0 0 0"/>
+        <axis xyz="0 0 0"/>
+    </joint>
 <!-- Base of Arm -->
-<link name="arm_base_link">
-    <inertial>
-        <mass value="0.1"/>
-        <origin rpy="0 0 0" xyz="0.0 0 0.0"/>
-        <inertia ixx="0.000041667" ixy="0" ixz="0" iyy="0.000041667" iyz="0" izz="0.000041667"/>
-    </inertial>
-    <collision>
-        <origin rpy="0 0 0" xyz="0 0 0"/>
-        <geometry>
-            <box size="0.05 0.05 0.05">
-        </geometry>
-    </collision>
-    <visual>
-        <origin rpy="0 0 0" xyz="0 0 0"/>
-        <geometry>
-            <box size="0.05 0.05 0.05">
-        </geometry>
-    </visual>
-</link>
+    <link name="arm_base_link">
+        <xacro:arm_base_inertial mass="${base_link_mass}"/>
+        <collision>
+            <origin rpy="0 0 0" xyz="0 0 0"/>
+            <geometry>
+                <box size="0.05 0.05 0.05"/>
+            </geometry>
+        </collision>
+        <visual>
+            <origin rpy="0 0 0" xyz="0 0 0"/>
+            <geometry>
+                <box size="0.05 0.05 0.05"/>
+            </geometry>
+            <material name="black">
+                <color rgba="0 0 0 1"/>
+            </material>
+        </visual>
+    </link>
+    <gazebo reference="arm_base_link">
+        <material>Gazebo/Black</material>
+    </gazebo>
 <!-- First Arm Link -->
-<link name="arm_link_01">
-    <inertial>
-        <mass value="0.025"/>
-        <origin rpy="0 0 0" xyz="0.0 0 0.0"/>
-        <inertia ixx="0.000010279" ixy="0" ixz="0" iyy="0.000010279" iyz="0" izz="0.000007225"/>
-    </inertial>
-    <collision>
-        <origin rpy="0 0 0" xyz="0 0 0"/>
-        <geometry>
-            <cylinder radius="0.017" length="0.04">
-        </geometry>
-    </collision>
-    <visual>
-        <origin rpy="0 0 0" xyz="0 0 0"/>
-        <geometry>
-            <cylinder radius="0.017" length="0.04">
-        </geometry>
-    </visual>
-</link>
-<joint name="arm_joint_1" type="revolute">
-    <axis xyz="0 0 1">
-    <limit effort="1000.0" lower="-3.14" upper="3.14" velocity="0.2"/>
-    <origin rpy="0 0 0" xyz="0 0 0.5"/>
-    <parent link="arm_base_link"/>
-    <child link="arm_link_01"/>
-</joint>
+    <link name="arm_link_01">
+        <xacro:link_inertial mass="${link_mass}"/>
+        <collision>
+            <origin rpy="0 0 0" xyz="0 0 0"/>
+            <geometry>
+                <cylinder radius="${arm_link_radius}" length="${arm_link_len}"/>
+            </geometry>
+        </collision>
+        <visual>
+            <origin rpy="0 0 0" xyz="0 0 0"/>
+            <geometry>
+                <cylinder radius="${arm_link_radius}" length="${arm_link_len}"/>
+            </geometry>
+            <material name="grey">
+                <color rgba="0.392 0.392 0.392 1"/>
+            </material>
+        </visual>
+    </link>
+    <joint name="arm_joint_1" type="revolute">
+        <axis xyz="0 0 1"/>
+        <limit effort="1000.0" lower="-3.14" upper="3.14" velocity="0.2"/>
+        <origin rpy="0 0 0" xyz="0 0 0.05"/>
+        <parent link="arm_base_link"/>
+        <child link="arm_link_01"/>
+    </joint>
+    <gazebo reference="arm_link_01">
+        <material>Gazebo/Grey</material>
+    </gazebo>
 <!-- Second Arm Link -->
-<link name="arm_link_02">
-    <inertial>
-        <mass value="0.025"/>
-        <origin rpy="0 0 0" xyz="0.0 0 0.0"/>
-        <inertia ixx="0.000010279" ixy="0" ixz="0" iyy="0.000010279" iyz="0" izz="0.000007225"/>
-    </inertial>
-    <collision>
+    <link name="arm_link_02">
+        <xacro:link_inertial mass="${link_mass}"/>
+        <collision>
+            <origin rpy="0 0 0" xyz="0 0 0.02"/>
+            <geometry>
+                <cylinder radius="${arm_link_radius}" length="${arm_link_len}"/>
+            </geometry>
+        </collision>
+        <visual>
+            <origin rpy="0 0 0" xyz="0 0 0.02"/>
+            <geometry>
+                <cylinder radius="${arm_link_radius}" length="${arm_link_len}"/>
+            </geometry>
+            <material name="grey">
+                <color rgba="0.392 0.392 0.392 1"/>
+            </material>
+        </visual>
+    </link>
+    <joint name="arm_joint_2" type="revolute">
+        <axis xyz="1 0 0"/>
+        <limit effort="1000.0" lower="-1.8" upper="1.8" velocity="0.2"/>
         <origin rpy="0 0 0" xyz="0 0 0.02"/>
-        <geometry>
-            <cylinder radius="0.017" length="0.04">
-        </geometry>
-    </collision>
-    <visual>
+        <parent link="arm_link_01"/>.000010279
+        <child link="arm_link_02"/>
+    </joint>
+    <gazebo reference="arm_link_02">
+        <material>Gazebo/Grey</material>
+    </gazebo>
+<!-- Third Arm Link -->
+    <link name="arm_link_03">
+        <xacro:link_inertial mass="${link_mass}"/>
+        <collision>
+            <origin rpy="0 0 0" xyz="0 0 0.04"/>
+            <geometry>
+                <cylinder radius="${arm_link_radius}" length="${arm_link_len}"/>
+            </geometry>
+        </collision>
+        <visual>
+            <origin rpy="0 0 0" xyz="0 0 0.04"/>
+            <geometry>
+                <cylinder radius="${arm_link_radius}" length="${arm_link_len}"/>
+            </geometry>
+            <material name="grey">
+                <color rgba="0.392 0.392 0.392 1"/>
+            </material>
+        </visual>
+    </link>
+    <joint name="arm_joint_3" type="revolute">
+        <axis xyz="1 0 0"/>
+        <limit effort="1000.0" lower="-1.8" upper="1.8" velocity="0.2"/>
         <origin rpy="0 0 0" xyz="0 0 0.02"/>
-        <geometry>
-            <cylinder radius="0.017" length="0.04">
-        </geometry>
-    </visual>
-</link>
-<joint name="arm_joint_2" type="revolute">
-    <axis xyz="1 0 0">
-    <limit effort="1000.0" lower="-1.8" upper="1.8" velocity="0.2"/>
-    <origin rpy="0 0 0" xyz="0 0 0.02"/>
-    <parent link="arm_link_01"/>
-    <child link="arm_link_02"/>
-</joint>
-<!-- Third Arm Link -->
-<link name="arm_link_03">
-    <inertial>
-        <mass value="0.025"/>
-        <origin rpy="0 0 0" xyz="0.0 0 0.0"/>
-        <inertia ixx="0.000010279" ixy="0" ixz="0" iyy="0.000010279" iyz="0" izz="0.000007225"/>
-    </inertial>
-    <collision>
+        <parent link="arm_link_02"/>
+        <child link="arm_link_03"/>
+    </joint>
+    <gazebo reference="arm_link_03">
+        <material>Gazebo/Grey</material>
+    </gazebo>
+<!-- Head Link -->
+    <link name="head_link">
+        <xacro:link_inertial mass="${link_mass}"/>
+        <collision>
+            <origin rpy="0 0 1.57" xyz="0 0 0.06"/>
+            <geometry>
+                <box size="${head_link_length} ${head_link_width} ${head_link_height}"/>
+            </geometry>
+        </collision>
+        <visual>
+            <origin rpy="0 0 1.57" xyz="0 0 0.06"/>
+            <geometry>
+                <box size="${head_link_length} ${head_link_width} ${head_link_height}"/>
+            </geometry>
+            <material name="black">
+                <color rgba="0 0 0 1"/>
+            </material>
+        </visual>
+    </link>
+    <joint name="head_joint" type="revolute">
+        <axis xyz="1 0 0"/>
+        <limit effort="1000.0" lower="-1.8" upper="1.8" velocity="0.5"/>
         <origin rpy="0 0 0" xyz="0 0 0.02"/>
-        <geometry>
-            <cylinder radius="0.017" length="0.04">
-        </geometry>
-    </collision>
-    <visual>
-        <origin rpy="0 0 0" xyz="0 0 0.02"/>
-        <geometry>
-            <cylinder radius="0.017" length="0.04">
-        </geometry>
-    </visual>
-</link>
-<joint name="arm_joint_3" type="revolute">
-    <axis xyz="1 0 0">
-    <limit effort="1000.0" lower="-1.8" upper="1.8" velocity="0.2"/>
-    <origin rpy="0 0 0" xyz="0 0 0.02"/>
-    <parent link="arm_link_02"/>
-    <child link="arm_link_03"/>
-</joint>
-<!-- Head Link -->
-<link name="head_link">
-    <inertial>
-        <mass value="0.025"/>
-        <origin rpy="0 0 0" xyz="0.0 0 0.0"/>
-        <inertia ixx="0.000010279" ixy="0" ixz="0" iyy="0.000010279" iyz="0" izz="0.000007225"/>
-    </inertial>
-    <collision>
-        <origin rpy="0 0 1.57" xyz="0 0 0.05"/>
-        <geometry>
-            <box size="0.017 0.094 0.84">
-        </geometry>
-    </collision>
-    <visual>
-        <origin rpy="0 0 1.57" xyz="0 0 0.05"/>
-        <geometry>
-            <box size="0.017 0.094 0.84">
-        </geometry>
-    </visual>
-</link>
-<joint name="head_joint" type="revolute">
-    <axis xyz="1 0 0">
-    <limit effort="1000.0" lower="-1.8" upper="1.8" velocity="0.5"/>
-    <origin rpy="0 0 1.57" xyz="0 0 0.05"/>
-    <parent link="arm_link_03"/>
-    <child link="arm_link_04"/>
-</joint>
+        <parent link="arm_link_03"/>
+        <child link="head_link"/>
+    </joint>
+    <gazebo reference="head_link">
+        <material>Gazebo/Black</material>
+    </gazebo>
 <!-- Gripper Link Right -->
-<link name="right_grip_link">
-    <inertial>
-        <mass value="0.01"/>
-        <origin xyz="0.0 0 0.0"/>
-        <inertia ixx="0.001" ixy="0" ixz="0" iyy="0.001" iyz="0" izz="0.001"/>
-    </inertial>
-    <collision>
-        <origin rpy="0 3.1415 -1.57" xyz="-0.32 0 0.06"/> <!-- 'x' value indicates aperture of gripper-->
-        <geometry>
-            <mesh filename="package://two_wheels_description/meshes/chain_link_grip_r.stl" scale="0.001 0.001 0.001"/>
-        </geometry>
-    </collision>
-    <visual>
-        <origin rpy="0 3.1415 -1.57" xyz="-0.32 0 0.06"/> <!-- 'x' value indicates aperture of gripper-->
-        <geometry>
-            <mesh filename="package://two_wheels_description/meshes/chain_link_grip_r.stl" scale="0.001 0.001 0.001"/>
-        </geometry>
-        <material name="grey"/>
-    </visual>
-</link>
-<joint name="right_grip_joint" type="prismatic">
-    <axis xyz="1 0 0">
-    <limit effort="1000.0" lower="-0.01" upper="0.035" velocity="6.5"/>
-    <origin rpy="0 0 0" xyz="-0.015 0 0.0"/>
-    <parent link="arm_link_04"/>
-    <child link="right_grip_link"/>
-</joint>
+    <link name="right_grip_link">
+        <xacro:gripper_inertial mass="${gripper_mass}"/>
+        <collision>
+            <origin rpy="0 3.1415 -1.57" xyz="-0.032 0 0.06"/> <!-- 'x' value indicates aperture of gripper-->
+            <geometry>
+                <!--Mesh obtained from  https://github.com/ROBOTIS-GIT/open_manipulator-->
+                <mesh filename="package://armbot_1/meshes/chain_link_grip_r.stl" scale="0.001 0.001 0.001"/>
+            </geometry>
+        </collision>
+        <visual>
+            <origin rpy="0 3.1415 -1.57" xyz="-0.032 0 0.06"/> <!-- 'x' value indicates aperture of gripper-->
+            <geometry>
+                <!--Mesh obtained from  https://github.com/ROBOTIS-GIT/open_manipulator-->
+                <mesh filename="package://armbot_1/meshes/chain_link_grip_r.stl" scale="0.001 0.001 0.001"/>
+            </geometry>
+            <material name="red">
+                <color rgba="1 0 0 1"/>
+            </material>
+        </visual>
+    </link>
+    <joint name="right_grip_joint" type="prismatic">
+        <axis xyz="1 0 0"/>
+        <limit effort="1000.0" lower="-0.01" upper="0.035" velocity="6.5"/>
+        <origin rpy="0 0 0" xyz="-0.015 0 0"/>
+        <parent link="head_link"/>
+        <child link="right_grip_link"/>
+    </joint>
+    <gazebo reference="right_grip_link">
+        <material>Gazebo/Red</material>
+    </gazebo>
 <!-- Gripper Link Left -->
-<link name="left_grip_link">
-    <inertial>
-        <mass value="0.01"/>
-        <origin xyz="0.0 0 0.0"/>
-        <inertia ixx="0.001" ixy="0" ixz="0" iyy="0.001" iyz="0" izz="0.001"/>
-    </inertial>
-    <collision>
-        <origin rpy="0 3.1415 -1.57" xyz="0.062 0 0.06"/> <!-- 'x' value indicates aperture of gripper-->
-        <geometry>
-            <mesh filename="package://two_wheels_description/meshes/chain_link_grip_l.stl" scale="0.001 0.001 0.001"/>
-        </geometry>
-    </collision>
-<xacro:property name="arm_link_radius" value="0.017"/>
-    <visual>
-        <origin rpy="0 3.1415 -1.57" xyz="0.062 0 0.06"/> <!-- 'x' value indicates aperture of gripper-->
-        <geometry>
-            <mesh filename="package://two_wheels_description/meshes/chain_link_grip_l.stl" scale="0.001 0.001 0.001"/>
-        </geometry>
-        <material name="grey"/>
-    </visual>
-</link>
-<joint name="left_grip_joint" type="prismatic">
-    <axis xyz="1 0 0">
-    <limit effort="1000.0" lower="-0.01" upper="0.035" velocity="6.5"/>
-    <origin rpy="0 0 0" xyz="-0.015 0 0.0"/>
-    <parent link="arm_link_04"/>
-    <child link="left_grip_link"/>
-</joint>
+    <link name="left_grip_link">
+        <xacro:gripper_inertial mass="${gripper_mass}"/>
+        <collision>
+            <origin rpy="0 3.1415 -1.57" xyz="0.062 0 0.06"/> <!-- 'x' value indicates aperture of gripper-->
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
File: src/diffbot_1/urdf/diffbot_2wheel.xacro (robot description, xacro)
@@ -1,43 +1,74 @@
 <?xml version="1.0"?>
 <robot name="diffbot_2wheel" xmlns:xacro="http://www.ros.org/wiki/xacro">
-<include filename="$(find erratic_description)/urdf/erratic_hokuyo_ laser.xacro" />
+<!--include filename="$(find erratic_description)/urdf/erratic_hokuyo_ laser.xacro"/-->
+<xacro:property name="chassis_length" value="0.2397125"/>
+<xacro:property name="chassis_width" value="0.1095375"/>
+<xacro:property name="chassis_height" value="0.0381"/>
+<xacro:property name="chassis_mass" value="1.3"/>
+<xacro:property name="caster_radius" value="0.03175"/>
+<xacro:property name="caster_length" value="0.0254"/>
 <xacro:property name="wheel_radius" value="0.03175"/>
 <xacro:property name="wheel_length" value="0.0254"/>
 <xacro:property name="wheel_mass" value="0.0283495"/>
-<xacro:property name="wheel_inertial_xx" value="0.000008668680579"/>
-<xacro:property name="wheel_inertial_yy" value="0.000008668680579"/>
-<xacro:property name="wheel_inertial_zz" value="0.000002381505654"/>
-<xacro:property name="wheel_x_pos" value="0.057546875"/>
-<xacro:property name="wheel_y_pos" value="0.04683125"/>
+<xacro:property name="wheel_x_pos" value="${chassis_length / 4}"/>
+<xacro:property name="wheel_y_pos" value="${(chassis_width / 2) + (wheel_length / 2)}"/>
 <xacro:property name="wheel_z_pos" value="0"/>
+<xacro:property name="caster_x_pos" value="${-(chassis_length / 4)}"/>
+<xacro:property name="caster_y_pos" value="0"/>
+<xacro:property name="caster_z_pos" value="0"/>
+<xacro:macro name="chassis_inertial" params="mass">
+    <inertial>
+        <mass value="${mass}"/>
+        <inertia ixx="${(1/12) * chassis_mass * ( (chassis_height * chassis_height) + (chassis_length * chassis_length)) }" ixy="0" ixz="0"
+                iyy="${(1/12) * chassis_mass * ( (chassis_width * chassis_width) + (chassis_height * chassis_height)) }" iyz="0"
+                izz="${(1/12) * chassis_mass * ( (chassis_width * chassis_width) + (chassis_length * chassis_length)) }"/>
+        </inertial>
+</xacro:macro>
+<xacro:macro name="wheel_inertial" params="mass">
+    <inertial>
+        <mass value="${mass}"/>
+        <inertia ixx="${(1/12) * wheel_mass * ( (3 * (wheel_radius * wheel_radius)) + (wheel_length * wheel_length)) }" ixy="0" ixz="0"
+                iyy="${(1/12) * wheel_mass * ( (3 * (wheel_radius * wheel_radius)) + (wheel_length * wheel_length)) }" iyz="0"
+                izz="${(1/2) * wheel_mass * (wheel_radius * wheel_radius) }"/>
+        </inertial>
+</xacro:macro>
 <!-- Hokuyo Laser -->
-<erratic_hokuyo_laser parent="base_link">
+<!--erratic_hokuyo_laser parent="base_link">
     <origin xyz="0.0 0.0 0.0381" rpy="0 0 0"/>
-</erratic_hokuyo_laser>
+</erratic_hokuyo_laser-->
 <!--Base Link-->
-    <link name="base_link">
-        <inertial>
-            <mass value="1.3"/>
-            <inertia ixx="0.006382316704" ixy="0" ixz="0"
-                    iyy="0.001457091340" iyz="0" izz="0.007524892544"/>
-        </inertial>
+    <link name="base_link"></link>
+    <joint name="base_to_chassis" type="fixed">
+        <parent link="base_link"/>
+        <child link="chassis_link"/>
+        <origin xyz="0 0 0" rpy="0 0 0"/>
+        <axis xyz="0 0 0"/>
+    </joint>
+<!--Chassis Link-->
+    <link name="chassis_link">
+        <xacro:chassis_inertial mass="${chassis_mass}"/>
         <collision name="base_link_collision">
             <geometry>
-                <box size="0.2397125 0.1095375 0.0381"/>
+                <box size="${chassis_length} ${chassis_width} ${chassis_height}"/>
             </geometry>
         </collision>
         <visual>
             <geometry>
-                <box size="0.2397125 0.1095375 0.0381"/>
+                <box size="${chassis_length} ${chassis_width} ${chassis_height}"/>
             </geometry>
-            <material name="bright_green">
-                <color rgba="0 255 0 1"/>
+            <material name="orange">
+                <color rgba="1 0.647 0 1"/>
             </material>
         </visual>
-        <!--Rear Caster-->
+    </link>
+    <gazebo reference="chassis_link">
+        <material>Gazebo/Orange</material>
+    </gazebo>
+<!--Rear Caster-->
+    <link name="caster_link">
         <collision name="caster_collision">
             <origin xyz="0 0 0" rpy="0 0 0"/>
             <geometry>
-                <cylinder radius="0.0" length="1.0"/>
+                <cylinder radius="${caster_radius}" length="${caster_length}"/>
             </geometry>
         </collision>
@@ -45,18 +76,23 @@
             <origin xyz="0 0 0" rpy="0 0 0"/>
             <geometry>
-                <cylinder radius="2.5625" length="1.0"/>
+                <cylinder radius="${caster_radius}" length="${caster_length}"/>
             </geometry>
-            <material name="bright_green">
-                <color rgba="0 255 0 1"/>
+            <material name="grey">
+                <color rgba="0.392 0.392 0.392 1"/>
             </material>
         </visual>
     </link>
+    <joint name="caster_joint" type="fixed">
+        <parent link="base_link"/>
+        <child link="caster_link"/>
+        <origin xyz="${caster_x_pos} ${caster_y_pos} ${caster_z_pos}" rpy="${pi/2} 0 0"/>
+        <axis xyz="0 0 0"/>
+    </joint>
+    <gazebo reference="caster_link">
+        <material>Gazebo/Grey</material>
+    </gazebo>
 <!--Right Wheel-->
     <link name="right_wheel">
-        <inertial>
-            <mass value="${wheel_mass}"/>
-            <inertia ixx="${wheel_inertial_xx}" ixy="0" ixz="0"
-                    iyy="${wheel_inertial_yy}" iyz="0" izz="${wheel_inertial_zz}"/>
-        </inertial>
+        <xacro:wheel_inertial mass="${wheel_mass}"/>
         <collision>
             <origin xyz="0 0 0" rpy="0 0 0"/>
@@ -78,14 +114,13 @@
         <parent link="base_link"/>
         <child link="right_wheel"/>
-        <origin xyz="${wheel_x_pos} ${wheel_y_pos} ${wheel_z_pos}" rpy="0 0 0"/>
-        <axis xyz="0 1 0"/>
+        <origin xyz="${wheel_x_pos} ${wheel_y_pos} ${wheel_z_pos}" rpy="${pi/2} 0 0"/>
+        <axis xyz="0 0 -1"/>
     </joint>
+    <gazebo reference="right_wheel">
+        <material>Gazebo/Black</material>
+    </gazebo>
 <!--Left Wheel-->
     <link name="left_wheel">
-        <inertial>
-            <mass value="${wheel_mass}"/>
-            <inertia ixx="${wheel_inertial_xx}" ixy="0" ixz="0"
-                    iyy="${wheel_inertial_yy}" iyz="0" izz="${wheel_inertial_zz}"/>
-        </inertial>
+        <xacro:wheel_inertial mass="${wheel_mass}"/>
         <collision>
             <origin xyz="0 0 0" rpy="0 0 0"/>
@@ -107,6 +142,9 @@
         <parent link="base_link"/>
         <child link="left_wheel"/>
-        <origin xyz="${wheel_x_pos} -${wheel_y_pos} ${wheel_z_pos}" rpy="0 0 0"/>
-        <axis xyz="0 1 0"/>
+        <origin xyz="${wheel_x_pos} -${wheel_y_pos} ${wheel_z_pos}" rpy="${pi/2} 0 0"/>
+        <axis xyz="0 0 1"/>
     </joint>
+    <gazebo reference="left_wheel">
+        <material>Gazebo/Black</material>
+    </gazebo>
 </robot>
