Commit message: Added Hokuyo sensors to differential models.

File: src/diffbot_1/urdf/diffbot2wheel_processed.urdf (robot description, URDF)
Before this commit: robot diffbot_2wheel, 5 links, 4 joints
Links:
- added link hokuyo_link, mass 1e-5; collision box size=0.1 0.1 0.1; visual mesh filename=package://diffbot_1/meshes/hokuyo.dae
Joints:
- added joint hokuyo_joint: type fixed, parent base_link, child hokuyo_link, origin xyz=0.059928125 0 0.0381 rpy=0 0 0, axis 0 1 0

File: src/diffbot_1/urdf/diffbot4wheel_processed.urdf (robot description, URDF)
Before this commit: robot diffbot_4wheel, 6 links, 5 joints
Links:
- added link hokuyo_link, mass 1e-5; collision box size=0.1 0.1 0.1; visual mesh filename=package://diffbot_1/meshes/hokuyo.dae
Joints:
- added joint hokuyo_joint: type fixed, parent base_link, child hokuyo_link, origin xyz=0 0 0.0492125 rpy=0 0 0, axis 0 1 0

File: src/diffbot_1/urdf/diffbot_2wheel.xacro (robot description, xacro)
@@ -1,5 +1,4 @@
 <?xml version="1.0"?>
 <robot name="diffbot_2wheel" xmlns:xacro="http://www.ros.org/wiki/xacro">
-<!--include filename="$(find erratic_description)/urdf/erratic_hokuyo_ laser.xacro"/-->
 <xacro:property name="chassis_length" value="0.2397125"/>
 <xacro:property name="chassis_width" value="0.1095375"/>
@@ -34,7 +33,65 @@
 </xacro:macro>
 <!-- Hokuyo Laser -->
-<!--erratic_hokuyo_laser parent="base_link">
-    <origin xyz="0.0 0.0 0.0381" rpy="0 0 0"/>
-</erratic_hokuyo_laser-->
+    <link name="hokuyo_link">
+        <collision>
+            <origin xyz="0 0 0" rpy="0 0 0"/>
+            <geometry>
+                <box size="0.1 0.1 0.1"/>
+            </geometry>
+        </collision>
+        <visual>
+            <origin xyz="0 0 0" rpy="0 0 0"/>
+            <geometry>
+                <!--Mesh obtained from  https://github.com/ros-simulation/gazebo_ros_demos-->
+                <mesh filename="package://diffbot_1/meshes/hokuyo.dae"/>
+            </geometry>
+        </visual>
+        <inertial>
+            <mass value="1e-5"/>
+            <origin xyz="0 0 0" rpy="0 0 0"/>
+            <inertia ixx="1e-6" ixy="0" ixz="0" iyy="1e-6" iyz="0" izz="1e-6" />
+        </inertial>
+    </link>
+    <joint name="hokuyo_joint" type="fixed">
+        <axis xyz="0 1 0" />
+        <origin xyz="${chassis_length / 4} 0 ${chassis_height}" rpy="0 0 0"/>
+        <parent link="base_link"/>
+        <child link="hokuyo_link"/>
+    </joint>
+    <!-- Gazebo Hokuyo -->
+    <gazebo reference="hokuyo_link">
+        <sensor type="gpu_ray" name="head_hokuyo_sensor">
+            <pose>0 0 0 0 0 0</pose>
+            <visualize>false</visualize>
+            <update_rate>40</update_rate>
+                <ray>
+                    <scan>
+                        <horizontal>
+                            <samples>720</samples>
+                            <resolution>1</resolution>
+                            <min_angle>-1.570796</min_angle>
+                            <max_angle>1.570796</max_angle>
+                        </horizontal>
+                    </scan>
+                    <range>
+                        <min>0.10</min>
+                        <max>30.0</max>
+                        <resolution>0.01</resolution>
+                    </range>
+                    <noise>
+                        <type>gaussian</type>
+                        <!-- Noise parameters based on published spec for Hokuyo laser achieving
+                        "+-30mm" accuracy at range < 10m. A mean of 0.0m and stddev of 0.01m will
+                        put 99.7% of samples within 0.03m of the true reading. -->
+                        <mean>0.0</mean>
+                        <stddev>0.01</stddev>
+                    </noise>
+                </ray>
+                <plugin name="gazebo_ros_head_hokuyo_controller" filename="libgazebo_ros_gpu_laser.so">
+                    <topicName>/rrbot/laser/scan</topicName>
+                    <frameName>hokuyo_link</frameName>
+                </plugin>
+        </sensor>
+    </gazebo>
 <!--Base Link-->
     <link name="base_link"></link>

File: src/diffbot_1/urdf/diffbot_4wheel.xacro (robot description, xacro)
@@ -1,5 +1,4 @@
 <?xml version="1.0"?>
 <robot name="diffbot_4wheel" xmlns:xacro="http://www.ros.org/wiki/xacro">
-<!--include filename="$(find erratic_description)/urdf/erratic_hokuyo_ laser.xacro"/ DEPRECATED-->
 <xacro:property name="chassis_length" value="0.2301875"/>
 <xacro:property name="chassis_width" value="0.0936625"/>
@@ -29,7 +28,65 @@
 </xacro:macro>
 <!-- Hokuyo Laser -->
-<!--erratic_hokuyo_laser parent="base_link">
-    <origin xyz="0.0 0.0 0.0" rpy="0 0 0"/>
-</erratic_hokuyo_laser-->
+    <link name="hokuyo_link">
+        <collision>
+            <origin xyz="0 0 0" rpy="0 0 0"/>
+            <geometry>
+                <box size="0.1 0.1 0.1"/>
+            </geometry>
+        </collision>
+        <visual>
+            <origin xyz="0 0 0" rpy="0 0 0"/>
+            <geometry>
+                <!--Mesh obtained from  https://github.com/ros-simulation/gazebo_ros_demos-->
+                <mesh filename="package://diffbot_1/meshes/hokuyo.dae"/>
+            </geometry>
+        </visual>
+        <inertial>
+            <mass value="1e-5"/>
+            <origin xyz="0 0 0" rpy="0 0 0"/>
+            <inertia ixx="1e-6" ixy="0" ixz="0" iyy="1e-6" iyz="0" izz="1e-6" />
+        </inertial>
+    </link>
+    <joint name="hokuyo_joint" type="fixed">
+        <axis xyz="0 1 0" />
+        <origin xyz="0 0 ${chassis_height}" rpy="0 0 0"/>
+        <parent link="base_link"/>
+        <child link="hokuyo_link"/>
+    </joint>
+    <!-- Gazebo Hokuyo -->
+    <gazebo reference="hokuyo_link">
+        <sensor type="gpu_ray" name="head_hokuyo_sensor">
+            <pose>0 0 0 0 0 0</pose>
+            <visualize>false</visualize>
+            <update_rate>40</update_rate>
+                <ray>
+                    <scan>
+                        <horizontal>
+                            <samples>720</samples>
+                            <resolution>1</resolution>
+                            <min_angle>-1.570796</min_angle>
+                            <max_angle>1.570796</max_angle>
+                        </horizontal>
+                    </scan>
+                    <range>
+                        <min>0.10</min>
+                        <max>30.0</max>
+                        <resolution>0.01</resolution>
+                    </range>
+                    <noise>
+                        <type>gaussian</type>
+                        <!-- Noise parameters based on published spec for Hokuyo laser achieving
+                        "+-30mm" accuracy at range < 10m. A mean of 0.0m and stddev of 0.01m will
+                        put 99.7% of samples within 0.03m of the true reading. -->
+                        <mean>0.0</mean>
+                        <stddev>0.01</stddev>
+                    </noise>
+                </ray>
+                <plugin name="gazebo_ros_head_hokuyo_controller" filename="libgazebo_ros_gpu_laser.so">
+                    <topicName>/rrbot/laser/scan</topicName>
+                    <frameName>hokuyo_link</frameName>
+                </plugin>
+        </sensor>
+    </gazebo>
 <!--Base Link-->
     <link name="base_link"></link>
