Commit message: Made some changes to the robot dimensions, mass, and gazebo plugin for caster wheel.

File: src/diffbot_1/urdf/diffbot2wheel_processed.urdf (robot description, URDF)
Before this commit: robot diffbot_2wheel, 6 links, 5 joints
Links:
- removed link chassis_link
- added link base_footprint
- link base_link: mass None -> 35; geometry collision box size=0.13 0.1095375 0.0381; visual box size=0.13 0.1095375 0.0381
- link caster_link: mass None -> 13; geometry collision sphere radius=0.02175; visual sphere radius=0.02175
- link left_wheel: mass 0.0283495 -> 0.1; geometry collision cylinder length=0.0254 radius=0.02175; visual cylinder length=0.0254 radius=0.02175
- link right_wheel: mass 0.0283495 -> 0.1; geometry collision cylinder length=0.0254 radius=0.02175; visual cylinder length=0.0254 radius=0.02175
Joints:
- removed joint base_to_chassis
- added joint base_footprint_to_base_link: type fixed, parent base_footprint, child base_link, origin xyz=0 0 0.02675 rpy=0 0 0, axis 0 0 0
- joint caster_joint: origin xyz=-0.059928125 0 0 rpy=1.5707963267948966 0 0 -> xyz=-0.0325 0 -0.01 rpy=0 0 0
- joint hokuyo_joint: origin xyz=0.059928125 0 0.0381 rpy=0 0 0 -> xyz=0.01625 0 0.0381 rpy=0 0 0
- joint joint_left_wheel: limit (none) -> effort=10000 velocity=1000; origin xyz=0.059928125 -0.06746875 0 rpy=1.5707963267948966 0 0 -> xyz=0.0325 0.06746875 -0.01 rpy=-1.5707963267948966 0 0
- joint joint_right_wheel: limit (none) -> effort=10000 velocity=1000; origin xyz=0.059928125 0.06746875 0 rpy=1.5707963267948966 0 0 -> xyz=0.0325 -0.06746875 -0.01 rpy=1.5707963267948966 0 0

File: src/diffbot_1/urdf/diffbot4wheel_processed.urdf (robot description, URDF)
Before this commit: robot diffbot_4wheel, 7 links, 6 joints
Links:
- removed link chassis_link
- added link base_footprint
- link back_left_wheel: mass 0.0283495 -> 0.1; geometry collision cylinder length=0.0127 radius=0.02175; visual cylinder length=0.0127 radius=0.02175
- link back_right_wheel: mass 0.0283495 -> 0.1; geometry collision cylinder length=0.0127 radius=0.02175; visual cylinder length=0.0127 radius=0.02175
- link base_link: mass None -> 25; geometry collision box size=0.16 0.0936625 0.0492125; visual box size=0.16 0.0936625 0.0492125
- link front_left_wheel: mass 0.0283495 -> 0.1; geometry collision cylinder length=0.0127 radius=0.02175; visual cylinder length=0.0127 radius=0.02175
- link front_right_wheel: mass 0.0283495 -> 0.1; geometry collision cylinder length=0.0127 radius=0.02175; visual cylinder length=0.0127 radius=0.02175
Joints:
- removed joint base_to_chassis
- added joint base_footprint_to_base_link: type fixed, parent base_footprint, child base_link, origin xyz=0 0 0.02675 rpy=0 0 0, axis 0 0 0
- joint joint_back_left_wheel: limit (none) -> effort=10000 velocity=1000; origin xyz=-0.057546875 -0.059531249999999994 0 rpy=-1.5707963267948966 0 0 -> xyz=-0.06175 0.05318125 -0.01 rpy=-1.5707963267948966 0 0
- joint joint_back_right_wheel: limit (none) -> effort=10000 velocity=1000; origin xyz=-0.057546875 0.059531249999999994 0 rpy=1.5707963267948966 0 0 -> xyz=-0.06175 -0.05318125 -0.01 rpy=1.5707963267948966 0 0
- joint joint_front_left_wheel: limit (none) -> effort=10000 velocity=1000; origin xyz=0.057546875 -0.059531249999999994 0 rpy=-1.5707963267948966 0 0 -> xyz=0.06175 0.05318125 -0.01 rpy=-1.5707963267948966 0 0
- joint joint_front_right_wheel: limit (none) -> effort=10000 velocity=1000; origin xyz=0.057546875 0.059531249999999994 0 rpy=1.5707963267948966 0 0 -> xyz=0.06175 -0.05318125 -0.01 rpy=1.5707963267948966 0 0

File: src/diffbot_1/urdf/diffbot_2wheel.xacro (robot description, xacro)
@@ -1,19 +1,24 @@
 <?xml version="1.0"?>
 <robot name="diffbot_2wheel" xmlns:xacro="http://www.ros.org/wiki/xacro">
-<xacro:property name="chassis_length" value="0.2397125"/>
+<!--Masses-->
+<xacro:property name="chassis_mass" value="35"/>
+<!--xacro:property name="wheel_mass" value="0.0283495"/-->
+<xacro:property name="wheel_mass" value="0.1"/>
+<xacro:property name="caster_mass" value="13"/>
+<!--Dimensions-->
+<xacro:property name="chassis_length" value="0.13"/>
 <xacro:property name="chassis_width" value="0.1095375"/>
 <xacro:property name="chassis_height" value="0.0381"/>
-<xacro:property name="chassis_mass" value="1.3"/>
-<xacro:property name="caster_radius" value="0.03175"/>
-<xacro:property name="caster_length" value="0.0254"/>
-<xacro:property name="wheel_radius" value="0.03175"/>
+<xacro:property name="caster_radius" value="0.02175"/>
+<xacro:property name="wheel_radius" value="0.02175"/>
 <xacro:property name="wheel_length" value="0.0254"/>
-<xacro:property name="wheel_mass" value="0.0283495"/>
+<!--Positions-->
 <xacro:property name="wheel_x_pos" value="${chassis_length / 4}"/>
 <xacro:property name="wheel_y_pos" value="${(chassis_width / 2) + (wheel_length / 2)}"/>
-<xacro:property name="wheel_z_pos" value="0"/>
+<xacro:property name="wheel_z_pos" value="-0.01"/>
 <xacro:property name="caster_x_pos" value="${-(chassis_length / 4)}"/>
 <xacro:property name="caster_y_pos" value="0"/>
-<xacro:property name="caster_z_pos" value="0"/>
+<xacro:property name="caster_z_pos" value="-0.01"/>
+<!--Inertial 1-->
 <xacro:macro name="chassis_inertial" params="mass">
     <inertial>
@@ -24,12 +29,141 @@
         </inertial>
 </xacro:macro>
-<xacro:macro name="wheel_inertial" params="mass">
+<!--Inertial 2-->
+<xacro:macro name="wheel_inertial" params="mass"> <!--True inertial measurements for wheels are too small, so they're substituted with 0.1-->
     <inertial>
         <mass value="${mass}"/>
-        <inertia ixx="${(1/12) * wheel_mass * ( (3 * (wheel_radius * wheel_radius)) + (wheel_length * wheel_length)) }" ixy="0" ixz="0"
-                iyy="${(1/12) * wheel_mass * ( (3 * (wheel_radius * wheel_radius)) + (wheel_length * wheel_length)) }" iyz="0"
-                izz="${(1/2) * wheel_mass * (wheel_radius * wheel_radius) }"/>
+        <inertia ixx="0.1" ixy="0" ixz="0"
+                iyy="0.1" iyz="0"
+                izz="0.1"/>
         </inertial>
 </xacro:macro>
+<!--Inertial 3-->0.1
+<xacro:macro name="caster_inertial" params="mass">
+    <inertial>
+        <mass value="${mass}"/>
+        <inertia ixx="${(2/5) * caster_mass * (caster_radius * caster_radius) }" ixy="0" ixz="0"
+                iyy="${(2/5) * caster_mass * (caster_radius * caster_radius) }" iyz="0"
+                izz="${(2/5) * caster_mass * (caster_radius * caster_radius) }"/>
+        </inertial>
+</xacro:macro>
+<!--Base Footprint-->
+    <link name="base_footprint"></link>
+    <joint name="base_footprint_to_base_link" type="fixed">
+        <parent link="base_footprint"/>
+        <child link="base_link"/>
+        <origin xyz="0 0 ${wheel_radius + 0.005}" rpy="0 0 0"/>
+        <axis xyz="0 0 0"/>
+    </joint>
+<!--Base Link-->
+    <link name="base_link">
+        <pose>0 0 0.1    0 0 0</pose> <!--Where to place robot in Gazebo-->
+        <xacro:chassis_inertial mass="${chassis_mass}"/>
+        <collision>
+            <geometry>
+                <box size="${chassis_length} ${chassis_width} ${chassis_height}"/>
+            </geometry>
+        </collision>
+        <visual>
+            <geometry>
+                <box size="${chassis_length} ${chassis_width} ${chassis_height}"/>
+            </geometry>
+            <material name="orange">
+                <color rgba="1 0.647 0 1"/>
+            </material>
+        </visual>
+    </link>
+    <gazebo reference="base_link">
+        <material>Gazebo/Orange</material>
+    </gazebo>
+<!--Rear Caster-->
+    <link name="caster_link">
+        <xacro:caster_inertial mass="${caster_mass}"/>
+        <collision>
+            <origin xyz="0 0 0" rpy="0 0 0"/>
+            <geometry>
+                <sphere radius="${caster_radius}"/>
+            </geometry>
+        </collision>
+        <visual>
+            <origin xyz="0 0 0" rpy="0 0 0"/>
+            <geometry>
+                <sphere radius="${caster_radius}"/>
+            </geometry>
+            <material name="grey">
+                <color rgba="0.392 0.392 0.392 1"/>
+            </material>
+        </visual>
+    </link>
+    <joint name="caster_joint" type="fixed">
+        <parent link="base_link"/>
+        <child link="caster_link"/>
+        <origin xyz="${caster_x_pos} ${caster_y_pos} ${caster_z_pos}" rpy="0 0 0"/>
+        <axis xyz="0 0 0"/>
+    </joint>
+    <gazebo reference="caster_link">
+        <mu1>0.0</mu1>
+        <mu2>0.0</mu2>
+        <material>Gazebo/Red</material>
+    </gazebo>
+<!--Right Wheel-->
+    <link name="right_wheel">
+        <xacro:wheel_inertial mass="${wheel_mass}"/>
+        <collision>
+            <origin xyz="0 0 0" rpy="0 0 0"/>
+            <geometry>
+                <cylinder radius="${wheel_radius}" length="${wheel_length}"/>
+            </geometry>
+        </collision>
+        <visual>
+            <origin xyz="0 0 0" rpy="0 0 0"/>
+            <geometry>
+                <cylinder radius="${wheel_radius}" length="${wheel_length}"/>
+            </geometry>
+            <material name="black">
+                <color rgba="0 0 0 1"/>
+            </material>
+        </visual>
+    </link>
+    <joint name="joint_right_wheel" type="continuous">
+        <parent link="base_link"/>
+        <child link="right_wheel"/>
+        <origin xyz="${wheel_x_pos} -${wheel_y_pos} ${wheel_z_pos}" rpy="${pi/2} 0 0"/>
+        <axis xyz="0 0 -1"/>
+        <limit effort="10000" velocity="1000"/>
+        <dynamics damping="1.0" friction="1.0"/>
+    </joint>
+    <gazebo reference="right_wheel">
+        <material>Gazebo/Black</material>
+    </gazebo>
+<!--Left Wheel-->
+    <link name="left_wheel">
+        <xacro:wheel_inertial mass="${wheel_mass}"/>
+        <collision>
+            <origin xyz="0 0 0" rpy="0 0 0"/>
+            <geometry>
+                <cylinder radius="${wheel_radius}" length="${wheel_length}"/>
+            </geometry>
+        </collision>
+        <visual>
+            <origin xyz="0 0 0" rpy="0 0 0"/>
+            <geometry>
+                <cylinder radius="${wheel_radius}" length="${wheel_length}"/>
+            </geometry>
+            <material name="black">
+                <color rgba="0 0 0 1"/>
+            </material>
+        </visual>
+    </link>
+    <joint name="joint_left_wheel" type="continuous">
+        <parent link="base_link"/>
+        <child link="left_wheel"/>
+        <origin xyz="${wheel_x_pos} ${wheel_y_pos} ${wheel_z_pos}" rpy="-${pi/2} 0 0"/>
+        <axis xyz="0 0 1"/>
+        <limit effort="10000" velocity="1000"/>
+        <dynamics damping="1.0" friction="1.0"/>
+    </joint>
+    <gazebo reference="left_wheel">
+        <material>Gazebo/Black</material>
+    </gazebo>
 <!-- Hokuyo Laser -->
     <link name="hokuyo_link">
@@ -55,13 +189,13 @@
     <joint name="hokuyo_joint" type="fixed">
         <axis xyz="0 1 0" />
-        <origin xyz="${chassis_length / 4} 0 ${chassis_height}" rpy="0 0 0"/>
+        <origin xyz="${chassis_length / 8} 0 ${chassis_height}" rpy="0 0 0"/>
         <parent link="base_link"/>
         <child link="hokuyo_link"/>
     </joint>
-    <!-- Gazebo Hokuyo -->
+<!-- Gazebo Hokuyo -->
     <gazebo reference="hokuyo_link">
-        <sensor type="gpu_ray" name="head_hokuyo_sensor">
+        <sensor type="ray" name="head_hokuyo_sensor">
             <pose>0 0 0 0 0 0</pose>
-            <visualize>false</visualize>
+            <visualize>true</visualize>
             <update_rate>40</update_rate>
                 <ray>
@@ -88,5 +222,5 @@
                     </noise>
                 </ray>
-                <plugin name="gazebo_ros_head_hokuyo_controller" filename="libgazebo_ros_gpu_laser.so">
+                <plugin name="gazebo_ros_head_hokuyo_controller" filename="libgazebo_ros_laser.so">
                     <topicName>/rrbot/laser/scan</topicName>
                     <frameName>hokuyo_link</frameName>
@@ -94,114 +228,19 @@
         </sensor>
     </gazebo>
-<!--Base Link-->
-    <link name="base_link"></link>
-    <joint name="base_to_chassis" type="fixed">
-        <parent link="base_link"/>
-        <child link="chassis_link"/>
-        <origin xyz="0 0 0" rpy="0 0 0"/>
-        <axis xyz="0 0 0"/>
-    </joint>
-<!--Chassis Link-->
-    <link name="chassis_link">
-        <xacro:chassis_inertial mass="${chassis_mass}"/>
-        <collision name="base_link_collision">
-            <geometry>
-                <box size="${chassis_length} ${chassis_width} ${chassis_height}"/>
-            </geometry>
-        </collision>
-        <visual>
-            <geometry>
-                <box size="${chassis_length} ${chassis_width} ${chassis_height}"/>
-            </geometry>
-            <material name="orange">
-                <color rgba="1 0.647 0 1"/>
-            </material>
-        </visual>
-    </link>
-    <gazebo reference="chassis_link">
-        <material>Gazebo/Orange</material>
-    </gazebo>
-<!--Rear Caster-->
-    <link name="caster_link">
-        <collision name="caster_collision">
-            <origin xyz="0 0 0" rpy="0 0 0"/>
-            <geometry>
-                <cylinder radius="${caster_radius}" length="${caster_length}"/>
-            </geometry>
-        </collision>
-        <visual>
-            <origin xyz="0 0 0" rpy="0 0 0"/>
-            <geometry>
-                <cylinder radius="${caster_radius}" length="${caster_length}"/>
-            </geometry>
-            <material name="grey">
-                <color rgba="0.392 0.392 0.392 1"/>
-            </material>
-        </visual>
-    </link>
-    <joint name="caster_joint" type="fixed">
-        <parent link="base_link"/>
-        <child link="caster_link"/>
-        <origin xyz="${caster_x_pos} ${caster_y_pos} ${caster_z_pos}" rpy="${pi/2} 0 0"/>
-        <axis xyz="0 0 0"/>
-    </joint>
-    <gazebo reference="caster_link">
-        <material>Gazebo/Grey</material>
-    </gazebo>
-<!--Right Wheel-->
-    <link name="right_wheel">
-        <xacro:wheel_inertial mass="${wheel_mass}"/>
-        <collision>
-            <origin xyz="0 0 0" rpy="0 0 0"/>
-            <geometry>
-                <cylinder radius="${wheel_radius}" length="${wheel_length}"/>
-            </geometry>
-        </collision>
-        <visual>
-            <origin xyz="0 0 0" rpy="0 0 0"/>
-            <geometry>
-                <cylinder radius="${wheel_radius}" length="${wheel_length}"/>
-            </geometry>
-            <material name="black">
-                <color rgba="0 0 0 1"/>
-            </material>
-        </visual>
-    </link>
-    <joint name="joint_right_wheel" type="continuous">
-        <parent link="base_link"/>
-        <child link="right_wheel"/>
-        <origin xyz="${wheel_x_pos} ${wheel_y_pos} ${wheel_z_pos}" rpy="${pi/2} 0 0"/>
-        <axis xyz="0 0 -1"/>
-    </joint>
-    <gazebo reference="right_wheel">
-        <material>Gazebo/Black</material>
-    </gazebo>
-<!--Left Wheel-->
-    <link name="left_wheel">
-        <xacro:wheel_inertial mass="${wheel_mass}"/>
-        <collision>
-            <origin xyz="0 0 0" rpy="0 0 0"/>
-            <geometry>
-                <cylinder radius="${wheel_radius}" length="${wheel_length}"/>
-            </geometry>
-        </collision>
-        <visual>
-            <origin xyz="0 0 0" rpy="0 0 0"/>
-            <geometry>
-                <cylinder radius="${wheel_radius}" length="${wheel_length}"/>
-            </geometry>
-            <material name="black">
-                <color rgba="0 0 0 1"/>
-            </material>
-        </visual>
-    </link>
-    <joint name="joint_left_wheel" type="continuous">
-        <parent link="base_link"/>
-        <child link="left_wheel"/>
-        <origin xyz="${wheel_x_pos} -${wheel_y_pos} ${wheel_z_pos}" rpy="${pi/2} 0 0"/>
-        <axis xyz="0 0 1"/>
-    </joint>
-    <gazebo reference="left_wheel">
-        <material>Gazebo/Black</material>
+<!--Gazebo Plugin-->
+    <gazebo>
+        <plugin name="differential_drive_controller" filename="libgazebo_ros_diff_drive.so">
+            <alwaysOn>true</alwaysOn>
+            <updateRate>20</updateRate>
+            <leftJoint>joint_left_wheel</leftJoint>
+            <rightJoint>joint_right_wheel</rightJoint>
+            <wheelSeparation>0.1095375</wheelSeparation>
+            <wheelDiameter>0.0635</wheelDiameter>
+            <torque>2.5</torque>
+            <commandTopic>cmd_vel</commandTopic>
+            <odometryTopic>odom</odometryTopic>
+            <odometryFrame>odom</odometryFrame>
+            <robotBaseFrame>base_footprint</robotBaseFrame>
+        </plugin>
     </gazebo>
 </robot>
